Commit message: added pose rewriter for AP DDS and refined robot_localization settings

File: urdf/lanealucys_robot.urdf (robot description, URDF)
Before this commit: robot lanealucys_robot, 2 links, 1 joints
Links:
- added link base_imu; visual box size=0.54 0.36 0.13
Joints:
- added joint base_to_imu: type fixed, parent base_link, child base_imu, origin xyz=0 0 0.03
